Commit message: Adjust URDF file: tune simulation dynamics and fix gripper joint
- Adjust inertial weights to improve simulation movements
- Update joint limits to reflect hardware constraints
- Use mimic joint for gripper jaws to ensure symmetrical opening and closing

File: hardware/elrobot/simulation/elrobot_follower.urdf (robot description, URDF)
Before this commit: robot Elrobot, 19 links, 18 joints
Links:
- link Gripper_Base_v1_1: mass 0.046895455343164964 -> 0.06244
- link Gripper_Gear_v1_1: mass 0.0024790841259162795 -> 0.0039
- link Gripper_Jaw_01_v1_1: mass 0.012492175356778453 -> 0.0125
- link Gripper_Jaw_02_v1_1: mass 0.012492175356778453 -> 0.0125
- link Joint_01_1: mass 0.036024842090469696 -> 0.05706
- link Joint_02_1: mass 0.04313419527395414 -> 0.05084
- link Joint_03_v1_1: mass 0.03705485612134295 -> 0.03822
- link Joint_04_v1_1: mass 0.04910540016805011 -> 0.05152
- link Joint_05_v1_1: mass 0.015030395597527186 -> 0.01756
- link Joint_06_v1_1: mass 0.03727709058376948 -> 0.03882
- link ST3215_1_v1_1: mass 0.03190666159632515 -> 0.055
- link ST3215_2_v1_1: mass 0.03190666159632515 -> 0.055
- link ST3215_3_v1_1: mass 0.03190666159632515 -> 0.055
- link ST3215_4_v1_1: mass 0.03190666159632515 -> 0.055
- link ST3215_5_v1_1: mass 0.03190666159632515 -> 0.055
- link ST3215_6_v1_1: mass 0.03190666159632515 -> 0.055
- link ST3215_7_v1_1: mass 0.03190666159632515 -> 0.055
- link ST3215_8_v1_1: mass 0.03190666159632515 -> 0.055
- link base_link: mass 0.06831242050694149 -> 0.03944
Joints:
- joint rev_motor_01: limit lower=-1.570796 upper=1.570796 effort=2.94 velocity=4.71 -> lower=-1.5509 upper=1.5509 effort=2.94 velocity=4.71
- joint rev_motor_02: limit lower=-1.570796 upper=1.570796 effort=2.94 velocity=4.71 -> lower=-1.6122 upper=1.6122 effort=2.94 velocity=4.71
- joint rev_motor_03: limit lower=-1.570796 upper=1.570796 effort=2.94 velocity=4.71 -> lower=-1.7610 upper=1.7610 effort=2.94 velocity=4.71
- joint rev_motor_04: limit lower=-1.570796 upper=1.570796 effort=2.94 velocity=4.71 -> lower=-1.7533 upper=1.7533 effort=2.94 velocity=4.71
- joint rev_motor_05: limit lower=-2.96706 upper=2.96706 effort=2.94 velocity=4.71 -> lower=-3.1907 upper=2.6998 effort=2.94 velocity=4.71
- joint rev_motor_06: limit lower=-1.570796 upper=1.570796 effort=2.94 velocity=4.71 -> lower=-1.3775 upper=1.7641 effort=2.94 velocity=4.71
- joint rev_motor_07: limit lower=-2.96706 upper=2.96706 effort=2.94 velocity=4.71 -> lower=-3.0710 upper=2.7796 effort=2.94 velocity=4.71
- joint rev_motor_08: limit lower=-1.48 upper=1.48 effort=2.94 velocity=4.71 -> lower=0 upper=2.2028 effort=2.94 velocity=4.71; type continuous -> revolute
- joint rev_motor_08_1: limit lower=-0.025 upper=0.0 effort=2.94 velocity=4.71 -> lower=-0.0255 upper=0.0 effort=2.94 velocity=4.71; mimic (none) -> joint=rev_motor_08 multiplier=-0.0115 offset=0
- joint rev_motor_08_2: limit lower=0.0 upper=0.025 effort=2.94 velocity=4.71 -> lower=0.0 upper=0.0255 effort=2.94 velocity=4.71; mimic (none) -> joint=rev_motor_08 multiplier=0.0115 offset=0; origin xyz=0.308573 -0.243367 -0.047491 rpy=0 0 0 -> xyz=0.308573 -0.243367 -0.049391 rpy=0 0 0

Commit message: Improve Joint 4, Joint 5 mechanical stopper to prevent it from breaking
- improve joints
- add missing Joint 4.stp file
- update limits for motor 5, motor 7 in urdf file
- update joint 5 and gripper position after auto-calibration

File: hardware/elrobot/simulation/elrobot_follower.urdf (robot description, URDF)
Before this commit: robot Elrobot, 19 links, 18 joints
Links:
- link Gripper_Base_v1_1: mass 0.06244 -> 0.046895455343164964
- link Gripper_Gear_v1_1: mass 0.0039 -> 0.0024790841259162795
- link Gripper_Jaw_01_v1_1: mass 0.0125 -> 0.012492175356778453
- link Gripper_Jaw_02_v1_1: mass 0.0125 -> 0.012492175356778453
- link Joint_01_1: mass 0.05706 -> 0.036024842090469696
- link Joint_02_1: mass 0.05084 -> 0.04313419527395414
- link Joint_03_v1_1: mass 0.03822 -> 0.03705485612134295
- link Joint_04_v1_1: mass 0.05152 -> 0.04910540016805011
- link Joint_05_v1_1: mass 0.01756 -> 0.015030395597527186
- link Joint_06_v1_1: mass 0.03882 -> 0.03727709058376948
- link ST3215_1_v1_1: mass 0.055 -> 0.03190666159632515
- link ST3215_2_v1_1: mass 0.055 -> 0.03190666159632515
- link ST3215_3_v1_1: mass 0.055 -> 0.03190666159632515
- link ST3215_4_v1_1: mass 0.055 -> 0.03190666159632515
- link ST3215_5_v1_1: mass 0.055 -> 0.03190666159632515
- link ST3215_6_v1_1: mass 0.055 -> 0.03190666159632515
- link ST3215_7_v1_1: mass 0.055 -> 0.03190666159632515
- link ST3215_8_v1_1: mass 0.055 -> 0.03190666159632515
- link base_link: mass 0.03944 -> 0.06831242050694149
Joints:
- joint rev_motor_05: limit lower=-3.1907 upper=2.6998 effort=2.94 velocity=4.71 -> lower=-2.62 upper=3.252 effort=2.94 velocity=4.71
- joint rev_motor_07: limit lower=-3.0710 upper=2.7796 effort=2.94 velocity=4.71 -> lower=-3.2014 upper=2.7336 effort=2.94 velocity=4.71

File: software/station/clients/station-viewer/public/elrobot/elrobot_follower.urdf (robot description, URDF)
Before this commit: robot Elrobot, 19 links, 18 joints
Joints:
- joint rev_motor_05: limit lower=-3.1907 upper=2.6998 effort=2.94 velocity=4.71 -> lower=-2.62 upper=3.252 effort=2.94 velocity=4.71
- joint rev_motor_07: limit lower=-3.0710 upper=2.7796 effort=2.94 velocity=4.71 -> lower=-3.2014 upper=2.7336 effort=2.94 velocity=4.71
